Commit message: urdf edition

File: car2/urdf/car2.urdf (robot description, URDF)
Before this commit: robot car2, 11 links, 10 joints
Joints:
- joint fin1: limit lower=-0.05 upper=0 effort=0 velocity=1.01 -> lower=-0.05 upper=0 effort=30.0 velocity=1.0
- joint fin2: limit lower=0 upper=0.05 effort=0 velocity=1.01 -> lower=0 upper=0.05 effort=30.0 velocity=1.0
- joint joint1: limit lower=-3.14 upper=3.14 effort=0 velocity=1.5 -> lower=-3.14 upper=3.14 effort=10.0 velocity=1.5
- joint joint2: limit lower=-0.2 upper=0 effort=0 velocity=1.5 -> lower=-0.2 upper=0 effort=50.0 velocity=1.5
- joint joint3: limit lower=-0.26 upper=0 effort=0 velocity=1.5 -> lower=-0.26 upper=0 effort=10.0 velocity=1.5
- joint joint4: limit lower=-1.57 upper=1.57 effort=0 velocity=1.5 -> lower=-1.57 upper=1.57 effort=10.0 velocity=1.5

Commit message: model updated

File: car2/urdf/car2.urdf (robot description, URDF)
Before this commit: robot car2, 11 links, 10 joints
Links:
- link base_link: mass 10.1 -> 10.782
- link castwheel: mass 1.957 -> 8.9511
- link leftwheel: mass 0.3096 -> 9.4472
- link link5: mass 1.748 -> 1.7726
- link rightwheel: mass 0.3096 -> 9.4472
Joints:
- joint castwheel_joint: axis 0.578881459990206 -0.0793276054052651 0.811543828945962 -> 0.57888 -0.079328 0.81154; origin xyz=-0.0164468565720474 -0.00527324448375706 -0.025 rpy=1.79986954685685 -0.424347021577185 0.792685410767129 -> xyz=0 -0.0012501 0.0925 rpy=1.7999 -0.42435 0.8825
- joint fin1: limit lower=-0.05 upper=0 effort=30.0 velocity=1.0 -> lower=-0.05 upper=0 effort=30 velocity=1.0
- joint fin2: limit lower=0 upper=0.05 effort=30.0 velocity=1.0 -> lower=0 upper=0.05 effort=30 velocity=1.0
- joint joint1: limit lower=-3.14 upper=3.14 effort=10.0 velocity=1.5 -> lower=-3.14 upper=3.14 effort=50 velocity=1.5; origin xyz=0 0 0.05 rpy=0 0 0 -> xyz=0 0 0.235 rpy=0 0 0.011375
- joint joint2: limit lower=-0.2 upper=0 effort=50.0 velocity=1.5 -> lower=-0.2 upper=0 effort=10 velocity=1.5; origin xyz=0 0 0.25 rpy=0 0 -0.078442 -> xyz=0 0 0.25 rpy=0 0 0
- joint joint3: limit lower=-0.26 upper=0 effort=10.0 velocity=1.5 -> lower=-0.26 upper=0 effort=10 velocity=1.5
- joint joint4: limit lower=-1.57 upper=1.57 effort=10.0 velocity=1.5 -> lower=-1.57 upper=1.57 effort=50 velocity=1.5
- joint joint5: limit lower=-3.14 upper=3.14 effort=0 velocity=1.5 -> lower=-3.14 upper=3.14 effort=50 velocity=1.5
- joint leftwheel_joint: origin xyz=0.055 -0.110423702246605 -0.035 rpy=-1.5707963267949 -0.105014840444308 3.14159265358979 -> xyz=0.057271 -0.19937 0.15 rpy=-1.5708 -0.10501 -3.1302
- joint rightwheel_joint: origin xyz=0.055 0.110423702246602 -0.035 rpy=1.5707963267949 -0.261061307663736 0 -> xyz=0.052721 0.20062 0.15 rpy=-1.5708 0.93928 -3.1302

Commit message: slam enabled

File: car2/urdf/car2.urdf (robot description, URDF)
Before this commit: robot car2, 11 links, 10 joints
Links:
- added link base_footprint
Joints:
- added joint base_joint: type fixed, parent base_link, child base_footprint, origin xyz=0.0 0.0 -0.15 rpy=0 0 0

Commit message: urdf file edited

File: car2/urdf/car2.urdf (robot description, URDF)
Before this commit: robot car2, 12 links, 11 joints
Links:
- added link arm_base_link
Joints:
- added joint arm_base_joint: type fixed, parent base_link, child arm_base_link, origin xyz=0 0 0.235 rpy=0 0 0
- joint fin2: mimic (none) -> joint=fin1 multiplier=-1 offset=0
- joint joint1: origin xyz=0 0 0.235 rpy=0 0 0.011375 -> xyz=0 0 0 rpy=0 0 0.011375; parent base_link -> arm_base_link
